File: Documentation/vrnding-mechine.brd (EAGLE design)
At the start: 160 x 100 mm, 43 parts, among them IC1 7805TV, IC2 REG1117

Commit message: test
Routing:
- net N$16: track 0.00 -> 160.0 mm
Other:
- board text added: "Tonday.INC"
Changed lines of the file:
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@@
 <?xml version="1.0" encoding="utf-8"?>
 <!DOCTYPE eagle SYSTEM "eagle.dtd">
-<eagle version="9.2.2">
+<eagle version="9.5.1">
 <drawing>
 <settings>
@@
 <wire x1="0" y1="0" x2="160" y2="0" width="0" layer="20"/>
 <wire x1="160" y1="0" x2="160" y2="100" width="0" layer="20"/>
-<wire x1="160" y1="100" x2="0" y2="100" width="0" layer="20"/>
 <wire x1="0" y1="100" x2="0" y2="0" width="0" layer="20"/>
+<text x="127" y="92.71" size="1.778" layer="16" rot="MR0">Tonday.INC</text>
 </plain>
 <attributes>
@@
 </polygon>
 </signal>
+<signal name="N$16">
+<wire x1="160" y1="100" x2="0" y2="100" width="0" layer="1"/>
+</signal>
 </signals>
